File: hardware/backplane/backplane.kicad_sch (KiCad schematic)
At the start: 35 parts, among them J1 Para o Mega (digital), J10 Slot 1, J11 Slot 2, J12 Slot 3, J13 Slot 4, J14 Slot 5, J15 Slot 6, J16 Slot 7, J17 Slot 8, J18 Slot 9, J19 Slot 10, J2 Para o Mega (analógico A0-A14), J20 Slot 11, J21 Slot 12, J3 Fonte externa 5 V

Commit message: Hardware: etiqueta com chave DIP para o Mega reconhecer cada módulo
- Módulos pequeno, médio e grande: mais um 74HC165 (U1) ligado a uma
  chave DIP de 8 vias, como primeiro byte de cada módulo na cadeia.
  Bits 7-6 dizem o tamanho da placa e 5-0 o número da seção, então o
  Mega percorre a fila sozinho, sem tabela de slots no firmware
- Os três módulos agora saem de um gerador só, com a mesma numeração
- Backplane: pull-down também no MISO, para o Mega ler "fim da fila"
  mesmo sem nenhum módulo; nota de que a ordem dos módulos não importa
- hardware/README.md: etiqueta, números e chaves DIP sugeridos para cada
  seção, teste de um módulo direto no Mega com 8 fios, ordem dos bytes
  e lista de peças atualizadas
- README: etiqueta na decisão de arquitetura, fase 2 e lista de compras

Co-Authored-By: Claude Opus 5.5 <noreply@anthropic.com>
Claude-Session: https://claude.ai/code/session_01XMhb4PzDFxzjZohaF3KBWg
Parts:
- added R22: 10k, Resistor_THT:R_Axial_DIN0207_L6.3mm_D2.5mm_P10.16mm_Horizontal, symbol Device:R
Connections:
- net C165_0: now also R22.1
- net GND: now also R22.2
