File: hardware/modulo_grande/modulo_grande.kicad_sch (KiCad schematic)
At the start: 37 parts, among them J1 Backplane (IDC 2x8), J2 Entradas 0-7, J3 Entradas 8-15, J4 Entradas 16-23, J5 LEDs 0-7, J6 LEDs 8-15, J7 Analógico (joystick, acelerad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, U1 74HC165, U2 74HC165, U3 74HC165, U4 74HC595, U5 74HC595

Commit message: Hardware: módulo pequeno (1 x 74HC165 + 1 x 74HC595) (#7)
* Roteiro: editor de nós de manobra na fase 4 e EXEC na fase 5

- Fase 4: 4 encoders (pró-grado, normal, radial, tempo) lidos por
  interrupção, botões NOVO/APAGAR/AP/PE/CIRC e dados do nó no LCD
- Fase 5: ARM + EXEC executa o nó de manobra
- Lista de compras: 6 encoders e os botões do editor

Co-Authored-By: Claude Opus 5.5 <noreply@anthropic.com>
Claude-Session: https://claude.ai/code/session_01XMhb4PzDFxzjZohaF3KBWg

* Hardware: esquemas KiCad do módulo genérico e do backplane

- hardware/modulo: placa igual para todas as seções do painel, com
  3 x 74HC165 (24 entradas com pull-up) e 2 x 74HC595 (16 saídas com
  resistor de LED), desacoplamento e conector IDC 2x8
- hardware/backplane: 12 slots IDC 2x8 encadeando os módulos no SPI do
  Mega, resistores de 47 ohms em série, pull-down no fim de cada cadeia,
  linhas analógicas dos slots 1 a 5 e jumper de alimentação
- PDFs dos esquemas ao lado de cada projeto
- hardware/README.md: pinagem do cabo, ligação ao Mega, regras dos slots,
  ordem dos bits para o firmware e lista de peças por placa
- README: painel em módulos com backplane como decisão de arquitetura;
  encoders lidos pela cadeia numa interrupção de timer

Co-Authored-By: Claude Opus 5.5 <noreply@anthropic.com>
Claude-Session: https://claude.ai/code/session_01XMhb4PzDFxzjZohaF3KBWg

* Hardware: módulo pequeno (1 x 74HC165 + 1 x 74HC595)

- hardware/modulo_pequeno: 8 entradas e 8 LEDs, mesmo cabo flat e mesmo
  slot do módulo grande, com o conector analógico
- hardware/modulo -> hardware/modulo_grande (24 entradas e 16 LEDs)
- hardware/README.md: qual placa vai em cada seção (6 pequenas e 6
  grandes), bytes de cada placa na cadeia, LEDs acesos só pelo estado
  do jogo e aviso sobre botões com LED de 5 V
- README: dois tamanhos de módulo na arquitetura, na fase 2 e na lista
  de compras

Co-Authored-By: Claude Opus 5.5 <noreply@anthropic.com>
Claude-Session: https://claude.ai/code/session_01XMhb4PzDF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
Other:
- note added: "Cadeia de entradas: SIN165 > U3 > U2 > U1 > SOUT165 (para o Mega). O Mega lê primeiro U1 (IN0-7), depois U2 (IN8-15), depois U3 (IN16-23). Botão ou chave: entre INn e GND. Apertado/ligado = 0 (pull-up de 10k). Cadeia de saídas: SIN595 > U4 > U5 > SOUT595 (para o próximo slot). LED: anodo em LEDn, catodo no GND. 1k limita a corrente a uns 3 mA, para os 8 LEDs de um 74HC595 ficarem abaixo de 70 mA.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"
- note added: "Módulo grande do painel"
- note added: "Para as seções com mais de 8 entradas ou mais de 8 LEDs (as outras usam o módulo pequeno). Monte sempre os 5 CIs: 24 entradas e 16 saídas para LED. Entrada ou saída sem uso fica livre."
- note removed: "Cadeia de entradas: SIN165 > U3 > U2 > U1 > SOUT165 (para o Mega). O Mega lê primeiro U1 (IN0-7), depois U2 (IN8-15), depois U3 (IN16-23). Botão ou chave: entre INn e GND. Apertado/ligado = 0 (pull-up de 10k). Cadeia de saídas: SIN595 > U4 > U5 > SOUT595 (para o próximo slot). LED: anodo em LEDn, catodo no GND. 1k limita a corrente a uns 3 mA, para os 8 LEDs de um 74HC595 ficarem abaixo de 70 mA."
- note removed: "Módulo genérico do painel"
- note removed: "Todos os módulos usam esta mesma placa, com todos os CIs montados: 24 entradas e 16 saídas para LED por módulo. Entrada ou saída sem uso fica livre."
- title: Módulo genérico do painel -> Módulo grande do painel

Commit message: Hardware: etiqueta com chave DIP para o Mega reconhecer cada módulo
- Módulos pequeno, médio e grande: mais um 74HC165 (U1) ligado a uma
  chave DIP de 8 vias, como primeiro byte de cada módulo na cadeia.
  Bits 7-6 dizem o tamanho da placa e 5-0 o número da seção, então o
  Mega percorre a fila sozinho, sem tabela de slots no firmware
- Os três módulos agora saem de um gerador só, com a mesma numeração
- Backplane: pull-down também no MISO, para o Mega ler "fim da fila"
  mesmo sem nenhum módulo; nota de que a ordem dos módulos não importa
- hardware/README.md: etiqueta, números e chaves DIP sugeridos para cada
  seção, teste de um módulo direto no Mega com 8 fios, ordem dos bytes
  e lista de peças atualizadas
- README: etiqueta na decisão de arquitetura, fase 2 e lista de compras

Co-Authored-By: Claude Opus 5.5 <noreply@anthropic.com>
Claude-Session: https://claude.ai/code/session_01XMhb4PzDFxzjZohaF3KBWg
Parts:
- removed C6: 10uF, Capacitor_THT:CP_Radial_D5.0mm_P2.00mm, symbol Device:C_Polarized
- removed U4: 74HC595, Package_DIP:DIP-16_W7.62mm_Socket, symbol 74xx:74HC595
- added C6: 100nF, Capacitor_THT:C_Disc_D5.0mm_W2.5mm_P5.00mm, symbol Device:C
- added C7: 10uF, Capacitor_THT:CP_Radial_D5.0mm_P2.00mm, symbol Device:C_Polarized
- added RN4: 10k, Resistor_THT:R_Array_SIP9, symbol Device:R_Network08
- added SW1: Etiqueta (DIP 8 vias), Button_Switch_THT:SW_DIP_SPSTx08_Slide_9.78x22.5mm_W7.62mm_P2.54mm, symbol Switch:SW_DIP_x08
- added U4: 74HC165, Package_DIP:DIP-16_W7.62mm_Socket, symbol 74xx:74HC165
- added U6: 74HC595, Package_DIP:DIP-16_W7.62mm_Socket, symbol 74xx:74HC595
Connections:
- net +5V: now also C6.1, C7.1, RN4.1 (common), U4.16 (VCC), U6.10 (~{SRCLR}), U6.16 (VCC)
- net CH595_1: now also U5.9 (QH'), U6.14 (SER); no longer U5.14 (SER)
- net GND: now also C6.2, C7.2, SW1.10, SW1.11, SW1.12, SW1.13, SW1.14, SW1.15, SW1.16, SW1.9, U4.15 (~{CE}), U4.8 (GND), U6.13 (~{OE}), U6.8 (GND)
- net IN0: now also RN2.2 (R1), U2.11 (D0); no longer RN1.2 (R1), U1.11 (D0)
- net IN1: now also RN2.3 (R2), U2.12 (D1); no longer RN1.3 (R2), U1.12 (D1)
- net IN10: now also RN3.4 (R3), U3.13 (D2); no longer RN2.4 (R3), U2.13 (D2)
- net IN11: now also RN3.5 (R4), U3.14 (D3); no longer RN2.5 (R4), U2.14 (D3)
- net IN12: now also RN3.6 (R5), U3.3 (D4); no longer RN2.6 (R5), U2.3 (D4)
- net IN13: now also RN3.7 (R6), U3.4 (D5); no longer RN2.7 (R6), U2.4 (D5)
- net IN14: now also RN3.8 (R7), U3.5 (D6); no longer RN2.8 (R7), U2.5 (D6)
- net IN15: now also RN3.9 (R8), U3.6 (D7); no longer RN2.9 (R8), U2.6 (D7)
- net IN16: now also RN4.2 (R1), U4.11 (D0); no longer RN3.2 (R1), U3.11 (D0)
- net IN17: now also RN4.3 (R2), U4.12 (D1); no longer RN3.3 (R2), U3.12 (D1)
- net IN18: now also RN4.4 (R3), U4.13 (D2); no longer RN3.4 (R3), U3.13 (D2)
- net IN19: now also RN4.5 (R4), U4.14 (D3); no longer RN3.5 (R4), U3.14 (D3)
- net IN2: now also RN2.4 (R3), U2.13 (D2); no longer RN1.4 (R3), U1.13 (D2)
- net IN20: now also RN4.6 (R5), U4.3 (D4); no longer RN3.6 (R5), U3.3 (D4)
- net IN21: now also RN4.7 (R6), U4.4 (D5); no longer RN3.7 (R6), U3.4 (D5)
- net IN22: now also RN4.8 (R7), U4.5 (D6); no longer RN3.8 (R7), U3.5 (D6)
- net IN23: now also RN4.9 (R8), U4.6 (D7); no longer RN3.9 (R8), U3.6 (D7)
- net IN3: now also RN2.5 (R4), U2.14 (D3); no longer RN1.5 (R4), U1.14 (D3)
- net IN4: now also RN2.6 (R5), U2.3 (D4); no longer RN1.6 (R5), U1.3 (D4)
- net IN5: now also RN2.7 (R6), U2.4 (D5); no longer RN1.7 (R6), U1.4 (D5)
- net IN6: now also RN2.8 (R7), U2.5 (D6); no longer RN1.8 (R7), U1.5 (D6)
- net IN7: now also RN2.9 (R8), U2.6 (D7); no longer RN1.9 (R8), U1.6 (D7)
- net IN8: now also RN3.2 (R1), U3.11 (D0); no longer RN2.2 (R1), U2.11 (D0)
- net IN9: now also RN3.3 (R2), U3.12 (D1); no longer RN2.3 (R2), U2.12 (D1)
- net OUT0: now also U5.15 (QA)
- net OUT1: now also U5.1 (QB)
- net OUT10: now also U6.2 (QC); no longer U5.2 (QC)
- net OUT11: now also U6.3 (QD); no longer U5.3 (QD)
- net OUT12: now also U6.4 (QE); no longer U5.4 (QE)
- net OUT13: now also U6.5 (QF); no longer U5.5 (QF)
- net OUT14: now also U6.6 (QG); no longer U5.6 (QG)
- net OUT15: now also U6.7 (QH); no longer U5.7 (QH)
- net OUT2: now also U5.2 (QC)
- net OUT3: now also U5.3 (QD)
- net OUT4: now also U5.4 (QE)
- net OUT5: now also U5.5 (QF)
- net OUT6: now also U5.6 (QG)
- net OUT7: now also U5.7 (QH)
- net OUT8: now also U6.15 (QA); no longer U5.15 (QA)
- net OUT9: now also U6.1 (QB); no longer U5.1 (QB)
- net PL: now also U4.1 (~{PL})
- net RCLK: now also U6.12 (RCLK)
- net SCK: now also U4.2 (CP), U6.11 (SRCLK)
- net SIN165: now also U4.10 (DS); no longer U3.10 (DS)
- net SIN595: now also U5.14 (SER)
- net SOUT595: now also U6.9 (QH'); no longer U5.9 (QH')
- new net CH165_3: U3.10 (DS), U4.9 (Q7)
- new net ID0: RN1.2 (R1), SW1.1, U1.11 (D0)
- new net ID1: RN1.3 (R2), SW1.2, U1.12 (D1)
- new net ID2: RN1.4 (R3), SW1.3, U1.13 (D2)
- new net ID3: RN1.5 (R4), SW1.4, U1.14 (D3)
- new net ID4: RN1.6 (R5), SW1.5, U1.3 (D4)
- new net ID5: RN1.7 (R6), SW1.6, U1.4 (D5)
- new net ID6: RN1.8 (R7), SW1.7, U1.5 (D6)
- new net ID7: RN1.9 (R8), SW1.8, U1.6 (D7)
- no-connect marks 3 -> 4
Other:
- note added: "Etiqueta"
- note added: "Etiqueta + 24 entradas + 16 saídas para LED. Monte sempre todos os CIs: a posição de cada byte na cadeia depende disso. Entrada ou saída sem uso fica livre."
- note added: "Etiqueta: chave k ligada (ON) = bit k-1 igual a 1. Bits 7-6 = tamanho (grande: 11); bits 5-0 = número da seção (1 a 62). Entradas: SIN165 > U4 > U3 > U2 > U1 > SOUT165 (para o Mega). O Mega lê nesta ordem: U1 (etiqueta), U2 (IN0-7), U3 (IN8-15), U4 (IN16-23). Botão ou chave: entre INn e GND. Apertado/ligado = 0 (pull-up de 10k). Saídas: SIN595 > U5 > U6 > SOUT595 (para o próximo slot). LED: anodo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"
- note added: "Um 100nF colado em cada CI"
- note removed: "Cadeia de entradas: SIN165 > U3 > U2 > U1 > SOUT165 (para o Mega). O Mega lê primeiro U1 (IN0-7), depois U2 (IN8-15), depois U3 (IN16-23). Botão ou chave: entre INn e GND. Apertado/ligado = 0 (pull-up de 10k). Cadeia de saídas: SIN595 > U4 > U5 > SOUT595 (para o próximo slot). LED: anodo em LEDn, catodo no GND. 1k limita a corrente a uns 3 mA, para os 8 LEDs de um 74HC595 ficarem abaixo de 70 mA.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"
- note removed: "Desacoplamento: um 100nF colado em cada CI"
- note removed: "Para as seções com mais de 8 entradas ou mais de 8 LEDs (as outras usam o módulo pequeno). Monte sempre os 5 CIs: 24 entradas e 16 saídas para LED. Entrada ou saída sem uso fica livre."
