File: hardware/modulo_medio/modulo_medio.kicad_sch (KiCad schematic)
At the start: 33 parts, among them J1 Backplane (IDC 2x8), J2 Entradas 0-7, J3 Entradas 8-15, J4 LEDs 0-7, J5 LEDs 8-15, J6 Analógico (joystick, acelerad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, U1 74HC165, U2 74HC165, U3 74HC595, U4 74HC595

Commit message: Hardware: etiqueta com chave DIP para o Mega reconhecer cada módulo
- Módulos pequeno, médio e grande: mais um 74HC165 (U1) ligado a uma
  chave DIP de 8 vias, como primeiro byte de cada módulo na cadeia.
  Bits 7-6 dizem o tamanho da placa e 5-0 o número da seção, então o
  Mega percorre a fila sozinho, sem tabela de slots no firmware
- Os três módulos agora saem de um gerador só, com a mesma numeração
- Backplane: pull-down também no MISO, para o Mega ler "fim da fila"
  mesmo sem nenhum módulo; nota de que a ordem dos módulos não importa
- hardware/README.md: etiqueta, números e chaves DIP sugeridos para cada
  seção, teste de um módulo direto no Mega com 8 fios, ordem dos bytes
  e lista de peças atualizadas
- README: etiqueta na decisão de arquitetura, fase 2 e lista de compras

Co-Authored-By: Claude Opus 5.5 <noreply@anthropic.com>
Claude-Session: https://claude.ai/code/session_01XMhb4PzDFxzjZohaF3KBWg
Parts:
- removed C5: 10uF, Capacitor_THT:CP_Radial_D5.0mm_P2.00mm, symbol Device:C_Polarized
- removed U3: 74HC595, Package_DIP:DIP-16_W7.62mm_Socket, symbol 74xx:74HC595
- added C5: 100nF, Capacitor_THT:C_Disc_D5.0mm_W2.5mm_P5.00mm, symbol Device:C
- added C6: 10uF, Capacitor_THT:CP_Radial_D5.0mm_P2.00mm, symbol Device:C_Polarized
- added RN3: 10k, Resistor_THT:R_Array_SIP9, symbol Device:R_Network08
- added SW1: Etiqueta (DIP 8 vias), Button_Switch_THT:SW_DIP_SPSTx08_Slide_9.78x22.5mm_W7.62mm_P2.54mm, symbol Switch:SW_DIP_x08
- added U3: 74HC165, Package_DIP:DIP-16_W7.62mm_Socket, symbol 74xx:74HC165
- added U5: 74HC595, Package_DIP:DIP-16_W7.62mm_Socket, symbol 74xx:74HC595
Connections:
- net +5V: now also C5.1, C6.1, RN3.1 (common), U3.16 (VCC), U5.10 (~{SRCLR}), U5.16 (VCC)
- net CH595_1: now also U4.9 (QH'), U5.14 (SER); no longer U4.14 (SER)
- net GND: now also C5.2, C6.2, SW1.10, SW1.11, SW1.12, SW1.13, SW1.14, SW1.15, SW1.16, SW1.9, U3.15 (~{CE}), U3.8 (GND), U5.13 (~{OE}), U5.8 (GND)
- net IN0: now also RN2.2 (R1), U2.11 (D0); no longer RN1.2 (R1), U1.11 (D0)
- net IN1: now also RN2.3 (R2), U2.12 (D1); no longer RN1.3 (R2), U1.12 (D1)
- net IN10: now also RN3.4 (R3), U3.13 (D2); no longer RN2.4 (R3), U2.13 (D2)
- net IN11: now also RN3.5 (R4), U3.14 (D3); no longer RN2.5 (R4), U2.14 (D3)
- net IN12: now also RN3.6 (R5), U3.3 (D4); no longer RN2.6 (R5), U2.3 (D4)
- net IN13: now also RN3.7 (R6), U3.4 (D5); no longer RN2.7 (R6), U2.4 (D5)
- net IN14: now also RN3.8 (R7), U3.5 (D6); no longer RN2.8 (R7), U2.5 (D6)
- net IN15: now also RN3.9 (R8), U3.6 (D7); no longer RN2.9 (R8), U2.6 (D7)
- net IN2: now also RN2.4 (R3), U2.13 (D2); no longer RN1.4 (R3), U1.13 (D2)
- net IN3: now also RN2.5 (R4), U2.14 (D3); no longer RN1.5 (R4), U1.14 (D3)
- net IN4: now also RN2.6 (R5), U2.3 (D4); no longer RN1.6 (R5), U1.3 (D4)
- net IN5: now also RN2.7 (R6), U2.4 (D5); no longer RN1.7 (R6), U1.4 (D5)
- net IN6: now also RN2.8 (R7), U2.5 (D6); no longer RN1.8 (R7), U1.5 (D6)
- net IN7: now also RN2.9 (R8), U2.6 (D7); no longer RN1.9 (R8), U1.6 (D7)
- net IN8: now also RN3.2 (R1), U3.11 (D0); no longer RN2.2 (R1), U2.11 (D0)
- net IN9: now also RN3.3 (R2), U3.12 (D1); no longer RN2.3 (R2), U2.12 (D1)
- net OUT0: now also U4.15 (QA)
- net OUT1: now also U4.1 (QB)
- net OUT10: now also U5.2 (QC); no longer U4.2 (QC)
- net OUT11: now also U5.3 (QD); no longer U4.3 (QD)
- net OUT12: now also U5.4 (QE); no longer U4.4 (QE)
- net OUT13: now also U5.5 (QF); no longer U4.5 (QF)
- net OUT14: now also U5.6 (QG); no longer U4.6 (QG)
- net OUT15: now also U5.7 (QH); no longer U4.7 (QH)
- net OUT2: now also U4.2 (QC)
- net OUT3: now also U4.3 (QD)
- net OUT4: now also U4.4 (QE)
- net OUT5: now also U4.5 (QF)
- net OUT6: now also U4.6 (QG)
- net OUT7: now also U4.7 (QH)
- net OUT8: now also U5.15 (QA); no longer U4.15 (QA)
- net OUT9: now also U5.1 (QB); no longer U4.1 (QB)
- net PL: now also U3.1 (~{PL})
- net RCLK: now also U5.12 (RCLK)
- net SCK: now also U3.2 (CP), U5.11 (SRCLK)
- net SIN165: now also U3.10 (DS); no longer U2.10 (DS)
- net SIN595: now also U4.14 (SER)
- net SOUT595: now also U5.9 (QH'); no longer U4.9 (QH')
- new net CH165_2: U2.10 (DS), U3.9 (Q7)
- new net ID0: RN1.2 (R1), SW1.1, U1.11 (D0)
- new net ID1: RN1.3 (R2), SW1.2, U1.12 (D1)
- new net ID2: RN1.4 (R3), SW1.3, U1.13 (D2)
- new net ID3: RN1.5 (R4), SW1.4, U1.14 (D3)
- new net ID4: RN1.6 (R5), SW1.5, U1.3 (D4)
- new net ID5: RN1.7 (R6), SW1.6, U1.4 (D5)
- new net ID6: RN1.8 (R7), SW1.7, U1.5 (D6)
- new net ID7: RN1.9 (R8), SW1.8, U1.6 (D7)
- no-connect marks 2 -> 3
Other:
- note added: "Etiqueta"
- note added: "Etiqueta + 16 entradas + 16 saídas para LED. Monte sempre todos os CIs: a posição de cada byte na cadeia depende disso. Entrada ou saída sem uso fica livre."
- note added: "Etiqueta: chave k ligada (ON) = bit k-1 igual a 1. Bits 7-6 = tamanho (médio: 10); bits 5-0 = número da seção (1 a 62). Entradas: SIN165 > U3 > U2 > U1 > SOUT165 (para o Mega). O Mega lê nesta ordem: U1 (etiqueta), U2 (IN0-7), U3 (IN8-15). Botão ou chave: entre INn e GND. Apertado/ligado = 0 (pull-up de 10k). Saídas: SIN595 > U4 > U5 > SOUT595 (para o próximo slot). LED: anodo em LEDn, catodo no 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"
- note added: "Um 100nF colado em cada CI"
- note removed: "Cadeia de entradas: SIN165 > U2 > U1 > SOUT165 (para o Mega). O Mega lê primeiro U1 (IN0-7), depois U2 (IN8-15). Botão ou chave: entre INn e GND. Apertado/ligado = 0 (pull-up de 10k). Cadeia de saídas: SIN595 > U3 > U4 > SOUT595 (para o próximo slot). LED: anodo em LEDn, catodo no GND. 1k limita a corrente a uns 3 mA, para os 8 LEDs de um 74HC595 ficarem abaixo de 70 mA. Quem acende os LEDs é o M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"
- note removed: "Desacoplamento: um 100nF colado em cada CI"
- note removed: "Para as seções com 9 a 16 entradas ou 9 a 16 LEDs. Monte sempre os 4 CIs: 16 entradas e 16 saídas para LED. Entrada ou saída sem uso fica livre."

Commit message: PCB do módulo médio: placa de 100 × 86 mm roteada, com Gerbers
- Placa de 2 camadas com furos M3 nos cantos, GND preenchido nas duas faces,
  trilhas de 0,3 mm nos sinais e 0,6 mm no +5V e GND. DRC sem erros e sem
  ligações faltando.
- hardware/pcb/modulo_medio.py gera a placa a partir do esquema: posiciona,
  roteia com o Freerouting, preenche o GND, roda o DRC e refaz os Gerbers.
- Gerbers e furação em hardware/modulo_medio/fabricacao/.
- Esquema: LEDs com 220 Ω, C6 de 470 µF (footprint de 10 mm) e resistores
  de 7,62 mm entre furos; PDF refeito.
- README do hardware: seção da PCB (como encomendar, montar e gerar de
  novo) e lista de peças atualizada.

Co-Authored-By: Claude Opus 5.5 <noreply@anthropic.com>
Claude-Session: https://claude.ai/code/session_01GYbCKeH4xeEesJ5HC66wNT
Parts:
- C6: value 10uF -> 470uF; footprint Capacitor_THT:CP_Radial_D5.0mm_P2.00mm -> Capacitor_THT:CP_Radial_D10.0mm_P5.00mm
- R1, R10, R11, R12, R13, R14, R15, R16, R2, R3, R4, R5, R6, R7, R8, R9: value 1k -> 220; footprint Resistor_THT:R_Axial_DIN0207_L6.3mm_D2.5mm_P10.16mm_Horizontal -> Resistor_THT:R_Axial_DIN0207_L6.3mm_D2.5mm_P7.62mm_Horizontal

Commit message: Módulo médio: 3 × 74HC595 e 12 jacks JST-XH para os korry (#45)
- Esquema: U6 (74HC595) no fim da cadeia de saída, com R17–R24 (220 Ω)
  e C7; as barras J2–J5 viram 12 jacks JST-XH de 4 vias (K1 a K12:
  GND, IN(k-1), LED(2k-2), LED(2k-1)) e uma barra J2 com IN12–IN15.
- PCB refeita em 100 × 100 mm: K1–K6 na borda de cima, K7–K12 na de
  baixo; DRC sem erros e sem ligações faltando; Gerbers novos.
- Documentação: tabelas do módulo médio, ordem dos bytes (3 de saída),
  lista de peças e a ficha do korry com os jacks.


Claude-Session: https://claude.ai/code/session_01GYbCKeH4xeEesJ5HC66wNT

Co-authored-by: Claude <noreply@anthropic.com>
Parts:
- removed J2: Entradas 0-7, Connector_PinHeader_2.54mm:PinHeader_1x10_P2.54mm_Vertical, symbol Connector_Generic:Conn_01x10
- removed J3: Entradas 8-15, Connector_PinHeader_2.54mm:PinHeader_1x10_P2.54mm_Vertical, symbol Connector_Generic:Conn_01x10
- removed J4: LEDs 0-7, Connector_PinHeader_2.54mm:PinHeader_1x10_P2.54mm_Vertical, symbol Connector_Generic:Conn_01x10
- removed J5: LEDs 8-15, Connector_PinHeader_2.54mm:PinHeader_1x10_P2.54mm_Vertical, symbol Connector_Generic:Conn_01x10
- added C7: 100nF, Capacitor_THT:C_Disc_D5.0mm_W2.5mm_P5.00mm, symbol Device:C
- added J2: Entradas 12-15, Connector_PinHeader_2.54mm:PinHeader_1x05_P2.54mm_Vertical, symbol Connector_Generic:Conn_01x05
- added K1: Korry 1, Connector_JST:JST_XH_B4B-XH-A_1x04_P2.50mm_Vertical, symbol Connector_Generic:Conn_01x04
- added K10: Korry 10, Connector_JST:JST_XH_B4B-XH-A_1x04_P2.50mm_Vertical, symbol Connector_Generic:Conn_01x04
- added K11: Korry 11, Connector_JST:JST_XH_B4B-XH-A_1x04_P2.50mm_Vertical, symbol Connector_Generic:Conn_01x04
- added K12: Korry 12, Connector_JST:JST_XH_B4B-XH-A_1x04_P2.50mm_Vertical, symbol Connector_Generic:Conn_01x04
- added K2: Korry 2, Connector_JST:JST_XH_B4B-XH-A_1x04_P2.50mm_Vertical, symbol Connector_Generic:Conn_01x04
- added K3: Korry 3, Connector_JST:JST_XH_B4B-XH-A_1x04_P2.50mm_Vertical, symbol Connector_Generic:Conn_01x04
- added K4: Korry 4, Connector_JST:JST_XH_B4B-XH-A_1x04_P2.50mm_Vertical, symbol Connector_Generic:Conn_01x04
- added K5: Korry 5, Connector_JST:JST_XH_B4B-XH-A_1x04_P2.50mm_Vertical, symbol Connector_Generic:Conn_01x04
- added K6: Korry 6, Connector_JST:JST_XH_B4B-XH-A_1x04_P2.50mm_Vertical, symbol Connector_Generic:Conn_01x04
- added K7: Korry 7, Connector_JST:JST_XH_B4B-XH-A_1x04_P2.50mm_Vertical, symbol Connector_Generic:Conn_01x04
- added K8: Korry 8, Connector_JST:JST_XH_B4B-XH-A_1x04_P2.50mm_Vertical, symbol Connector_Generic:Conn_01x04
- added K9: Korry 9, Connector_JST:JST_XH_B4B-XH-A_1x04_P2.50mm_Vertical, symbol Connector_Generic:Conn_01x04
- added R17, R18, R19, R20, R21, R22, R23, R24: 220, Resistor_THT:R_Axial_DIN0207_L6.3mm_D2.5mm_P7.62mm_Horizontal, symbol Device:R
- added U6: 74HC595, Package_DIP:DIP-16_W7.62mm_Socket, symbol 74xx:74HC595
Connections:
- net +5V: now also C7.1, U6.10 (~{SRCLR}), U6.16 (VCC)
- net GND: now also C7.2, J2.5 (Pin_5), K1.1 (Pin_1), K10.1 (Pin_1), K11.1 (Pin_1), K12.1 (Pin_1), K2.1 (Pin_1), K3.1 (Pin_1), K4.1 (Pin_1), K5.1 (Pin_1), K6.1 (Pin_1), K7.1 (Pin_1), K8.1 (Pin_1), K9.1 (Pin_1), U6.13 (~{OE}), U6.8 (GND)
- net IN0: now also K1.2 (Pin_2)
- net IN1: now also K2.2 (Pin_2)
- net IN10: now also K11.2 (Pin_2)
- net IN11: now also K12.2 (Pin_2)
- net IN12: now also J2.1 (Pin_1)
- net IN13: now also J2.2 (Pin_2)
- net IN14: now also J2.3 (Pin_3)
- net IN15: now also J2.4 (Pin_4)
- net IN2: now also K3.2 (Pin_2)
- net IN3: now also K4.2 (Pin_2)
- net IN4: now also K5.2 (Pin_2)
- net IN5: now also K6.2 (Pin_2)
- net IN6: now also K7.2 (Pin_2)
- net IN7: now also K8.2 (Pin_2)
- net IN8: now also K9.2 (Pin_2)
- net IN9: now also K10.2 (Pin_2)
- net LED0: now also K1.3 (Pin_3)
- net LED1: now also K1.4 (Pin_4)
- net LED10: now also K6.3 (Pin_3)
- net LED11: now also K6.4 (Pin_4)
- net LED12: now also K7.3 (Pin_3)
- net LED13: now also K7.4 (Pin_4)
- net LED14: now also K8.3 (Pin_3)
- net LED15: now also K8.4 (Pin_4)
- net LED2: now also K2.3 (Pin_3)
- net LED3: now also K2.4 (Pin_4)
- net LED4: now also K3.3 (Pin_3)
- net LED5: now also K3.4 (Pin_4)
- net LED6: now also K4.3 (Pin_3)
- net LED7: now also K4.4 (Pin_4)
- net LED8: now also K5.3 (Pin_3)
- net LED9: now also K5.4 (Pin_4)
- net RCLK: now also U6.12 (RCLK)
- net SCK: now also U6.11 (SRCLK)
- net SOUT595: now also U6.9 (QH'); no longer U5.9 (QH')
- new net CH595_2: U5.9 (QH'), U6.14 (SER)
- new net LED16: K9.3 (Pin_3), R17.2
- new net LED17: K9.4 (Pin_4), R18.2
- new net LED18: K10.3 (Pin_3), R19.2
- new net LED19: K10.4 (Pin_4), R20.2
- new net LED20: K11.3 (Pin_3), R21.2
- new net LED21: K11.4 (Pin_4), R22.2
- new net LED22: K12.3 (Pin_3), R23.2
- new net LED23: K12.4 (Pin_4), R24.2
- new net OUT16: R17.1, U6.15 (QA)
- new net OUT17: R18.1, U6.1 (QB)
- new net OUT18: R19.1, U6.2 (QC)
- new net OUT19: R20.1, U6.3 (QD)
- new net OUT20: R21.1, U6.4 (QE)
- new net OUT21: R22.1, U6.5 (QF)
- new net OUT22: R23.1, U6.6 (QG)
- new net OUT23: R24.1, U6.7 (QH)
Other:
- note added: "Etiqueta + 16 entradas + 24 saídas para LED. Monte sempre todos os CIs: a posição de cada byte na cadeia depende disso. Entrada ou saída sem uso fica livre."
- note added: "Etiqueta: chave k ligada (ON) = bit k-1 igual a 1. Bits 7-6 = tamanho (médio: 10); bits 5-0 = número da seção (1 a 62). Entradas: SIN165 > U3 > U2 > U1 > SOUT165 (para o Mega). O Mega lê nesta ordem: U1 (etiqueta), U2 (IN0-7), U3 (IN8-15). Botão ou chave: entre INn e GND. Apertado/ligado = 0 (pull-up de 10k). Saídas: SIN595 > U4 > U5 > U6 > SOUT595 (para o próximo slot). LED: anodo em LEDn, catod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"
- note added: "Korry (K1 a K12, JST-XH de 4 vias) Kk: 1 GND, 2 IN(k-1), 3 LED(2k-2) em cima, 4 LED(2k-1) embaixo. J2: IN12 a IN15, para botões comuns."
- note removed: "Etiqueta + 16 entradas + 16 saídas para LED. Monte sempre todos os CIs: a posição de cada byte na cadeia depende disso. Entrada ou saída sem uso fica livre."
- note removed: "Etiqueta: chave k ligada (ON) = bit k-1 igual a 1. Bits 7-6 = tamanho (médio: 10); bits 5-0 = número da seção (1 a 62). Entradas: SIN165 > U3 > U2 > U1 > SOUT165 (para o Mega). O Mega lê nesta ordem: U1 (etiqueta), U2 (IN0-7), U3 (IN8-15). Botão ou chave: entre INn e GND. Apertado/ligado = 0 (pull-up de 10k). Saídas: SIN595 > U4 > U5 > SOUT595 (para o próximo slot). LED: anodo em LEDn, catodo no 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"
- moved on the sheet: R1, R10, R11, R12, R13, R14, R15, R16, R2, R3, R4, R5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
